File: pcb/Nucleo64STLinkShield.kicad_pcb (KiCad board)
At the start: 4 copper layers, 44 x 24.6 mm, 7 parts, among them J1 SWD, J2 Debug, J3 UART, J4 USB Power, J5 Nucleo-64 ST-Link Selector

Commit message: Added nets for the pin sockets.
Parts:
- moved J4 2.49 mm to (158.1, 92.6), turned to -90 degrees
Connections:
- J1 pad 1: unconnected-(J1-Pin_1-Pad1) -> +3.3V
- J1 pad 2: unconnected-(J1-Pin_2-Pad2) -> swclk
- J1 pad 3: unconnected-(J1-Pin_3-Pad3) -> GND
- J1 pad 4: unconnected-(J1-Pin_4-Pad4) -> swdio
- J1 pad 5: unconnected-(J1-Pin_5-Pad5) -> RESET
- J1 pad 6: unconnected-(J1-Pin_6-Pad6) -> swo
- J3 pad 1: unconnected-(J3-Pin_1-Pad1) -> stlink_rx
- J3 pad 2: unconnected-(J3-Pin_2-Pad2) -> stlink_tx
- J4 pad 1: unconnected-(J4-Pin_1-Pad1) -> +3.3V
Changed lines of the file:
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@@
 	(net 7 "swo")
 	(net 8 "stlink_rx")
-	(net 9 "unconnected-(J1-Pin_2-Pad2)")
-	(net 10 "unconnected-(J1-Pin_1-Pad1)")
-	(net 11 "unconnected-(J1-Pin_6-Pad6)")
-	(net 12 "unconnected-(J1-Pin_4-Pad4)")
-	(net 13 "unconnected-(J1-Pin_5-Pad5)")
-	(net 14 "unconnected-(J1-Pin_3-Pad3)")
-	(net 15 "unconnected-(J3-Pin_1-Pad1)")
-	(net 16 "unconnected-(J3-Pin_2-Pad2)")
-	(net 17 "unconnected-(J4-Pin_2-Pad2)")
-	(net 18 "unconnected-(J4-Pin_1-Pad1)")
-	(net 19 "unconnected-(J5-Pin_2-Pad2)")
-	(net 20 "unconnected-(J5-Pin_1-Pad1)")
-	(net 21 "unconnected-(J5-Pin_3-Pad3)")
-	(net 22 "unconnected-(J5-Pin_4-Pad4)")
+	(net 9 "unconnected-(J4-Pin_2-Pad2)")
+	(net 10 "unconnected-(J5-Pin_2-Pad2)")
+	(net 11 "unconnected-(J5-Pin_1-Pad1)")
+	(net 12 "unconnected-(J5-Pin_3-Pad3)")
+	(net 13 "unconnected-(J5-Pin_4-Pad4)")
 	(footprint "LOGO"
 		(locked yes)
@@
 			(layers "*.Cu" "*.Mask")
 			(remove_unused_layers no)
-			(net 20 "unconnected-(J5-Pin_1-Pad1)")
+			(net 11 "unconnected-(J5-Pin_1-Pad1)")
 			(pinfunction "Pin_1")
-			(pintype "passive")
+			(pintype "passive+no_connect")
 		)
 		(pad "2" thru_hole circle
@@
 			(layers "*.Cu" "*.Mask")
 			(remove_unused_layers no)
-			(net 19 "unconnected-(J5-Pin_2-Pad2)")
+			(net 10 "unconnected-(J5-Pin_2-Pad2)")
 			(pinfunction "Pin_2")
-			(pintype "passive")
+			(pintype "passive+no_connect")
 		)
 		(pad "3" thru_hole circle
@@
 			(layers "*.Cu" "*.Mask")
 			(remove_unused_layers no)
-			(net 21 "unconnected-(J5-Pin_3-Pad3)")
+			(net 12 "unconnected-(J5-Pin_3-Pad3)")
 			(pinfunction "Pin_3")
-			(pintype "passive")
+			(pintype "passive+no_connect")
 		)
 		(pad "4" thru_hole circle
@@
 			(layers "*.Cu" "*.Mask")
 			(remove_unused_layers no)
-			(net 22 "unconnected-(J5-Pin_4-Pad4)")
+			(net 13 "unconnected-(J5-Pin_4-Pad4)")
 			(pinfunction "Pin_4")
-			(pintype "passive")
+			(pintype "passive+no_connect")
 		)
 		(embedded_fonts no)
@@
 			(layers "*.Cu" "*.Mask")
 			(remove_unused_layers no)
-			(net 10 "unconnected-(J1-Pin_1-Pad1)")
+			(net 2 "+3.3V")
 			(pinfunction "Pin_1")
 			(pintype "passive")
@@
 			(layers "*.Cu" "*.Mask")
 			(remove_unused_layers no)
-			(net 9 "unconnected-(J1-Pin_2-Pad2)")
+			(net 5 "swclk")
 			(pinfunction "Pin_2")
 			(pintype "passive")
@@
 			(layers "*.Cu" "*.Mask")
 			(remove_unused_layers no)
-			(net 14 "unconnected-(J1-Pin_3-Pad3)")
+			(net 1 "GND")
 			(pinfunction "Pin_3")
 			(pintype "passive")
@@
 			(layers "*.Cu" "*.Mask")
 			(remove_unused_layers no)
-			(net 12 "unconnected-(J1-Pin_4-Pad4)")
+			(net 4 "swdio")
 			(pinfunction "Pin_4")
 			(pintype "passive")
@@
 			(layers "*.Cu" "*.Mask")
 			(remove_unused_layers no)
-			(net 13 "unconnected-(J1-Pin_5-Pad5)")
+			(net 3 "RESET")
 			(pinfunction "Pin_5")
 			(pintype "passive")
@@
 			(layers "*.Cu" "*.Mask")
 			(remove_unused_layers no)
-			(net 11 "unconnected-(J1-Pin_6-Pad6)")
+			(net 7 "swo")
 			(pinfunction "Pin_6")
 			(pintype "passive")
@@
 		(locked yes)
 		(layer "B.Cu")
-		(at 160.55 92.675 90)
+		(at 158.06 92.6 -90)
 		(descr "Through hole straight socket strip, 1x02, 2.54mm pitch, single row (from Kicad 4.0.7), script generated")
 		(tags "Through hole socket strip THT 1x02 2.54mm single row")
@@
 		(attr through_hole)
 		(fp_line
+			(start 0 1.33)
+			(end 1.33 1.33)
+			(stroke
+				(width 0.12)
+				(type solid)
+			)
+			(layer "B.SilkS")
+		)
+		(fp_line
+			(start 1.33 1.33)
+			(end 1.33 0)
+			(stroke
+				(width 0.12)
+				(type solid)
+			)
+			(layer "B.SilkS")
+		)
+		(fp_line
+			(start -1.33 -1.27)
+			(end 1.33 -1.27)
+			(stroke
+				(width 0.12)
+				(type solid)
+			)
+			(layer "B.SilkS")
+		)
+		(fp_line
+			(start -1.33 -1.27)
+			(end -1.33 -3.87)
+			(stroke
+				(width 0.12)
+				(type solid)
+			)
+			(layer "B.SilkS")
+		)
+		(fp_line
+			(start 1.33 -1.27)
+			(end 1.33 -3.87)
+			(stroke
+				(width 0.12)
+				(type solid)
+			)
+			(layer "B.SilkS")
+		)
+		(fp_line
 			(start -1.33 -3.87)
 			(end 1.33 -3.87)
@@
 		)
 		(fp_line
-			(start 1.33 -1.27)
-			(end 1.33 -3.87)
-			(stroke
-				(width 0.12)
-				(type solid)
-			)
-			(layer "B.SilkS")
-		)
-		(fp_line
-			(start -1.33 -1.27)
-			(end -1.33 -3.87)
-			(stroke
-				(width 0.12)
-				(type solid)
-			)
-			(layer "B.SilkS")
-		)
-		(fp_line
-			(start -1.33 -1.27)
-			(end 1.33 -1.27)
-			(stroke
-				(width 0.12)
-				(type solid)
-			)
-			(layer "B.SilkS")
-		)
-		(fp_line
-			(start 1.33 1.33)
-			(end 1.33 0)
-			(stroke
-				(width 0.12)
-				(type solid)
-			)
-			(layer "B.SilkS")
-		)
-		(fp_line
-			(start 0 1.33)
-			(end 1.33 1.33)
-			(stroke
-				(width 0.12)
-				(type solid)
-			)
-			(layer "B.SilkS")
+			(start -1.8 1.8)
+			(end 1.75 1.8)
+			(stroke
+				(width 0.05)
+				(type solid)
+			)
+			(layer "B.CrtYd")
+		)
+		(fp_line
+			(start 1.75 1.8)
+			(end 1.75 -4.3)
+			(stroke
+				(width 0.05)
+				(type solid)
+			)
+			(layer "B.CrtYd")
+		)
+		(fp_line
+			(start -1.8 -4.3)
+			(end -1.8 1.8)
+			(stroke
+				(width 0.05)
+				(type solid)
+			)
+			(layer "B.CrtYd")
 		)
 		(fp_line
@@
 		)
 		(fp_line
-			(start -1.8 -4.3)
-			(end -1.8 1.8)
-			(stroke
-				(width 0.05)
-				(type solid)
-			)
-			(layer "B.CrtYd")
-		)
-		(fp_line
-			(start 1.75 1.8)
-			(end 1.75 -4.3)
-			(stroke
-				(width 0.05)
-				(type solid)
-			)
-			(layer "B.CrtYd")
-		)
-		(fp_line
-			(start -1.8 1.8)
-			(end 1.75 1.8)
-			(stroke
-				(width 0.05)
-				(type solid)
-			)
-			(layer "B.CrtYd")
+			(start -1.27 1.27)
+			(end 0.635 1.27)
+			(stroke
+				(width 0.1)
+				(type solid)
+			)
+			(layer "B.Fab")
+		)
+		(fp_line
+			(start 0.635 1.27)
+			(end 1.27 0.635)
+			(stroke
+				(width 0.1)
+				(type solid)
+			)
+			(layer "B.Fab")
+		)
+		(fp_line
+			(start 1.27 0.635)
+			(end 1.27 -3.81)
+			(stroke
+				(width 0.1)
+				(type solid)
+			)
+			(layer "B.Fab")
+		)
+		(fp_line
+			(start -1.27 -3.81)
+			(end -1.27 1.27)
+			(stroke
+				(width 0.1)
+				(type solid)
+			)
+			(layer "B.Fab")
 		)
 		(fp_line
@@
 			(layer "B.Fab")
 		)
-		(fp_line
-			(start -1.27 -3.81)
-			(end -1.27 1.27)
-			(stroke
-				(width 0.1)
-				(type solid)
-			)
-			(layer "B.Fab")
-		)
-		(fp_line
-			(start 1.27 0.635)
-			(end 1.27 -3.81)
-			(stroke
-				(width 0.1)
-				(type solid)
-			)
-			(layer "B.Fab")
-		)
-		(fp_line
-			(start 0.635 1.27)
-			(end 1.27 0.635)
-			(stroke
-				(width 0.1)
-				(type solid)
-			)
-			(layer "B.Fab")
-		)
-		(fp_line
-			(start -1.27 1.27)
-			(end 0.635 1.27)
-			(stroke
-				(width 0.1)
-				(type solid)
-			)
-			(layer "B.Fab")
-		)
 		(fp_text user "${REFERENCE}"
 			(at 0 -1.27 0)
@@
 		)
 		(pad "1" thru_hole rect
-			(at 0 0 90)
+			(at 0 0 270)
 			(size 1.7 1.7)
 			(drill 1)
 			(layers "*.Cu" "*.Mask")
 			(remove_unused_layers no)
-			(net 18 "unconnected-(J4-Pin_1-Pad1)")
+			(net 2 "+3.3V")
 			(pinfunction "Pin_1")
 			(pintype "passive")
 		)
 		(pad "2" thru_hole circle
-			(at 0 -2.54 90)
+			(at 0 -2.54 270)
 			(size 1.7 1.7)
 			(drill 1)
 			(layers "*.Cu" "*.Mask")
 			(remove_unused_layers no)
-			(net 17 "unconnected-(J4-Pin_2-Pad2)")
+			(net 9 "unconnected-(J4-Pin_2-Pad2)")
 			(pinfunction "Pin_2")
-			(pintype "passive")
+			(pintype "passive+no_connect")
 		)
 		(embedded_fonts no)
@@
 			(layers "*.Cu" "*.Mask")
 			(remove_unused_layers no)
-			(net 15 "unconnected-(J3-Pin_1-Pad1)")
+			(net 8 "stlink_rx")
 			(pinfunction "Pin_1")
 			(pintype "passive")
@@
 			(layers "*.Cu" "*.Mask")
 			(remove_unused_layers no)
-			(net 16 "unconnected-(J3-Pin_2-Pad2)")
+			(net 6 "stlink_tx")
 			(pinfunction "Pin_2")
 			(pintype "passive")

Commit message: Added supporting components.
Parts:
- added D2: GREEN, LED_SMD:LED_1206_3216Metric_Pad1.42x1.75mm_HandSolder, F.Cu at (147.2, 106.4)
- added J6: Conn_01x06, Connector_PinHeader_2.54mm:PinHeader_1x03_P2.54mm_Vertical, F.Cu at (128.8, 93.7)
- added J7: Conn_01x06, Connector_PinHeader_2.54mm:PinHeader_1x03_P2.54mm_Vertical, F.Cu at (128.8, 106.3)
- added R1: 1k, Resistor_SMD:R_1206_3216Metric_Pad1.30x1.75mm_HandSolder, F.Cu at (164.2, 97.8)
- added R30: 2K, Resistor_SMD:R_1206_3216Metric_Pad1.30x1.75mm_HandSolder, F.Cu at (147.2, 111.6)
- added SW2: B3U-1000P, Button_Switch_SMD:SW_SPST_B3U-1000P, F.Cu at (159.2, 97.8)
- moved G*** 2.80 mm to (159.2, 105.6)
Other:
- board text added: "+3.3V"
- board text added: "GND"
- board text added: "RESET"
