File: pcb/PowerDistributionSystem_Stepper_Motor_Driver_TMC2209.kicad_sch (KiCad schematic)
At the start: 16 parts, among them U4 TMC2209-LA-T

Commit message: Laid TMC2209 stepper motor drivers out.
Parts:
- C8: value 25TGV100M8X10.5 -> 865080343009; footprint Capacitor_SMD:CP_Elec_8x10.5 -> Capacitor_SMD:CP_Elec_6.3x5.4
- U4: footprint Package_DFN_QFN:VQFN-28-1EP_5x5mm_P0.5mm_EP3.7x3.7mm_ThermalVias -> pcb:VQFN-28-1EP_5x5mm_P0.5mm_EP3.7x3.7mm_ThermalVias
Changed lines of the file:
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@@
 			)
 		)
-		(property "Value" "25TGV100M8X10.5"
+		(property "Value" "865080343009"
 			(at 223.52 87.63 0)
 			(effects
@@
 			)
 		)
-		(property "Footprint" "Capacitor_SMD:CP_Elec_8x10.5"
+		(property "Footprint" "Capacitor_SMD:CP_Elec_6.3x5.4"
 			(at 220.6752 90.17 0)
 			(effects
@@
 			)
 		)
-		(property "Footprint" "Package_DFN_QFN:VQFN-28-1EP_5x5mm_P0.5mm_EP3.7x3.7mm_ThermalVias"
+		(property "Footprint" "pcb:VQFN-28-1EP_5x5mm_P0.5mm_EP3.7x3.7mm_ThermalVias"
 			(at 134.62 153.67 0)
 			(effects

Commit message: Added regulators for burn-wire.
Parts:
- U4: footprint pcb:VQFN-28-1EP_5x5mm_P0.5mm_EP3.7x3.7mm_ThermalVias -> Package_DFN_QFN:VQFN-28-1EP_5x5mm_P0.5mm_EP3.7x3.7mm_ThermalVias
- renumbered JP2 to JP3, JP3 to JP4
