File: pcb/VehiclePowerDistributionSystem.kicad_pcb (KiCad board)
At the start: 4 copper layers, 70 x 70 mm, 66 parts, among them J1 B2B-XH-A, J10 FFC2B28-24-G, J2 B2B-XH-A, J3 B2B-XH-A, J4 B4B-XH-A, J5 B4B-XH-A, J6 B4B-XH-A, J7 B8B-XH-A, U2 D24V7F5, U3 D24V7F3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

Commit message: `Vehicle PDS I/O (V1 : Fixed pin-count).`
Parts:
- renumbered J10 to J8
Connections:
- J8 pad 10: +5V -> GND
- J8 pad 11: GND -> +5V
- J8 pad 12: +3.3V -> GND
- J8 pad 13: GND -> +3.3V
- J8 pad 14: +5V -> GND
- J8 pad 15: GND -> +5V
- J8 pad 16: EXTERNAL_DETECTED -> GND
- J8 pad 17: BATTERY_ALLOWED -> EXTERNAL_DETECTED
- J8 pad 18: +3.3V -> BATTERY_ALLOWED
- J8 pad 19: MOTOR_DIR_Z -> +3.3V
- J8 pad 2: MOTOR_STEP_X -> GND
- J8 pad 20: MOTOR_DIR_Y -> MOTOR_DIR_Z
- J8 pad 21: MOTOR_DIR_X -> MOTOR_DIR_Y
- J8 pad 22: GND -> MOTOR_DIR_X
- J8 pad 23: (no net) -> GND
- J8 pad 24: (no net) -> GND
- J8 pad 3: MOTOR_STEP_Y -> MOTOR_STEP_X
- J8 pad 4: MOTOR_STEP_Z -> MOTOR_STEP_Y
- J8 pad 5: +3.3V -> MOTOR_STEP_Z
- J8 pad 6: MOTOR_DISABLE -> +3.3V
- J8 pad 7: MOTOR_UART_RX -> MOTOR_DISABLE
- J8 pad 8: MOTOR_UART_TX -> MOTOR_UART_RX
- J8 pad 9: GND -> MOTOR_UART_TX
Changed lines of the file:
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@@
 		(at 117.5 100 90)
 		(descr "FFC/FPC connector, 24 top-side contacts, 0.5mm pitch, SMT")
-		(property "Reference" "J10"
+		(property "Reference" "J8"
 			(at 0 3.11 90)
 			(layer "B.SilkS")
@@
 			)
 		)
-		(property "Description" "Generic connector, single row, 01x22, script generated (kicad-library-utils/schlib/autogen/connector/)"
+		(property "Description" "Generic connector, single row, 01x24, script generated (kicad-library-utils/schlib/autogen/connector/)"
 			(at 0 0 90)
 			(layer "B.Fab")
@@
 			(size 0.3 1.1)
 			(layers "B.Cu" "B.Mask" "B.Paste")
-			(net 10 "MOTOR_STEP_X")
+			(net 1 "GND")
 			(pinfunction "Pin_2")
 			(pintype "passive")
@@
 			(size 0.3 1.1)
 			(layers "B.Cu" "B.Mask" "B.Paste")
-			(net 48 "MOTOR_STEP_Y")
+			(net 10 "MOTOR_STEP_X")
 			(pinfunction "Pin_3")
 			(pintype "passive")
@@
 			(size 0.3 1.1)
 			(layers "B.Cu" "B.Mask" "B.Paste")
-			(net 49 "MOTOR_STEP_Z")
+			(net 48 "MOTOR_STEP_Y")
 			(pinfunction "Pin_4")
 			(pintype "passive")
@@
 			(size 0.3 1.1)
 			(layers "B.Cu" "B.Mask" "B.Paste")
-			(net 2 "+3.3V")
+			(net 49 "MOTOR_STEP_Z")
 			(pinfunction "Pin_5")
 			(pintype "passive")
@@
 			(size 0.3 1.1)
 			(layers "B.Cu" "B.Mask" "B.Paste")
-			(net 6 "MOTOR_DISABLE")
+			(net 2 "+3.3V")
 			(pinfunction "Pin_6")
 			(pintype "passive")
@@
 			(size 0.3 1.1)
 			(layers "B.Cu" "B.Mask" "B.Paste")
-			(net 8 "MOTOR_UART_RX")
+			(net 6 "MOTOR_DISABLE")
 			(pinfunction "Pin_7")
 			(pintype "passive")
@@
 			(size 0.3 1.1)
 			(layers "B.Cu" "B.Mask" "B.Paste")
-			(net 9 "MOTOR_UART_TX")
+			(net 8 "MOTOR_UART_RX")
 			(pinfunction "Pin_8")
 			(pintype "passive")
@@
 			(size 0.3 1.1)
 			(layers "B.Cu" "B.Mask" "B.Paste")
-			(net 1 "GND")
+			(net 9 "MOTOR_UART_TX")
 			(pinfunction "Pin_9")
 			(pintype "passive")
@@
 			(size 0.3 1.1)
 			(layers "B.Cu" "B.Mask" "B.Paste")
-			(net 53 "+5V")
+			(net 1 "GND")
 			(pinfunction "Pin_10")
 			(pintype "passive")
@@
 			(size 0.3 1.1)
 			(layers "B.Cu" "B.Mask" "B.Paste")
-			(net 1 "GND")
+			(net 53 "+5V")
 			(pinfunction "Pin_11")
 			(pintype "passive")
@@
 			(size 0.3 1.1)
 			(layers "B.Cu" "B.Mask" "B.Paste")
-			(net 2 "+3.3V")
+			(net 1 "GND")
 			(pinfunction "Pin_12")
 			(pintype "passive")
@@
 			(size 0.3 1.1)
 			(layers "B.Cu" "B.Mask" "B.Paste")
-			(net 1 "GND")
+			(net 2 "+3.3V")
 			(pinfunction "Pin_13")
 			(pintype "passive")
@@
 			(size 0.3 1.1)
 			(layers "B.Cu" "B.Mask" "B.Paste")
-			(net 53 "+5V")
+			(net 1 "GND")
 			(pinfunction "Pin_14")
 			(pintype "passive")
@@
 			(size 0.3 1.1)
 			(layers "B.Cu" "B.Mask" "B.Paste")
-			(net 1 "GND")
+			(net 53 "+5V")
 			(pinfunction "Pin_15")
 			(pintype "passive")
@@
 			(size 0.3 1.1)
 			(layers "B.Cu" "B.Mask" "B.Paste")
-			(net 55 "EXTERNAL_DETECTED")
+			(net 1 "GND")
 			(pinfunction "Pin_16")
 			(pintype "passive")
@@
 			(size 0.3 1.1)
 			(layers "B.Cu" "B.Mask" "B.Paste")
-			(net 54 "BATTERY_ALLOWED")
+			(net 55 "EXTERNAL_DETECTED")
 			(pinfunction "Pin_17")
 			(pintype "passive")
@@
 			(size 0.3 1.1)
 			(layers "B.Cu" "B.Mask" "B.Paste")
-			(net 2 "+3.3V")
+			(net 54 "BATTERY_ALLOWED")
 			(pinfunction "Pin_18")
 			(pintype "passive")
@@
 			(size 0.3 1.1)
 			(layers "B.Cu" "B.Mask" "B.Paste")
-			(net 51 "MOTOR_DIR_Z")
+			(net 2 "+3.3V")
 			(pinfunction "Pin_19")
 			(pintype "passive")
@@
 			(size 0.3 1.1)
 			(layers "B.Cu" "B.Mask" "B.Paste")
-			(net 50 "MOTOR_DIR_Y")
+			(net 51 "MOTOR_DIR_Z")
 			(pinfunction "Pin_20")
 			(pintype "passive")
@@
 			(size 0.3 1.1)
 			(layers "B.Cu" "B.Mask" "B.Paste")
-			(net 13 "MOTOR_DIR_X")
+			(net 50 "MOTOR_DIR_Y")
 			(pinfunction "Pin_21")
 			(pintype "passive")
@@
 			(size 0.3 1.1)
 			(layers "B.Cu" "B.Mask" "B.Paste")
-			(net 1 "GND")
+			(net 13 "MOTOR_DIR_X")
 			(pinfunction "Pin_22")
 			(pintype "passive")
@@
 			(size 0.3 1.1)
 			(layers "B.Cu" "B.Mask" "B.Paste")
+			(net 1 "GND")
+			(pinfunction "Pin_23")
+			(pintype "passive")
 		)
 		(pad "24" smd rect
@@
 			(size 0.3 1.1)
 			(layers "B.Cu" "B.Mask" "B.Paste")
+			(net 1 "GND")
+			(pinfunction "Pin_24")
+			(pintype "passive")
 		)
 		(embedded_fonts no)
