File: pcb/VehiclePowerDistributionSystem.kicad_pcb (KiCad board)
At the start: 4 copper layers, 70 x 70 mm, 70 parts, among them J1 B4B-XH-A, J2 B4B-XH-A, J3 B4B-XH-A, J4 B8B-XH-A, J5 XF3M_2415_1B, J6 B2B-XH-A, J7 B2B-XH-A, J8 B2B-XH-A, U1 TMC2209-LA-T, U2 TMC2209-LA-T, U3 TMC2209-LA-T, U4 BTS462TATMA1, U5 D24V7F5, U6 D24V7F3

Commit message: Finalized `VPDS-R2`.
Parts:
- R4: value 1k -> 100
- R5: value 47k -> 1k
- moved R14 0.30 mm to (127.3, 125.8)
Other:
- board text added: "+"
- board text added: "+11V"
- board text added: "+EXTERNAL"
- board text added: "-"
- board text added: "B2-B1-A2-A1 YEL-ORG-BLU-RED"
- board text added: "UART"
- board text added: "VPDS-R2"
- board text added: "WASTE PRODUCT OF PHUC DOAN"
- board text removed: "VPDS-R1"
Changed lines of the file:
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@@
 			)
 		)
-		(property "Value" "1k"
+		(property "Value" "100"
 			(at 0 1.83 90)
 			(layer "F.Fab")
@@
 			)
 		)
-		(property "Value" "47k"
+		(property "Value" "1k"
 			(at 0 1.83 90)
 			(layer "F.Fab")
@@
 		(tags "resistor handsolder")
 		(property "Reference" "R1"
-			(at 0 -1.83 180)
+			(at -3.2 0 180)
 			(layer "F.SilkS")
 			(effects
@@
 		(tags "resistor handsolder")
 		(property "Reference" "R16"
-			(at 0 -1.7 0)
+			(at -3.7 -0.1 0)
 			(layer "F.SilkS")
 			(effects
@@
 		(tags "connector JST XH vertical")
 		(property "Reference" "J8"
-			(at 1.25 3.55 180)
+			(at -3.8 2.275 180)
 			(layer "B.SilkS")
 			(effects
@@
 		(tags "connector JST XH vertical")
 		(property "Reference" "J6"
-			(at 1.25 3.55 180)
+			(at -3.800001 2.275 180)
 			(layer "B.SilkS")
 			(effects
@@
 	(footprint "Resistor_SMD:R_1206_3216Metric_Pad1.30x1.75mm_HandSolder"
 		(layer "B.Cu")
-		(at 127.6 125.85 90)
+		(at 127.3 125.85 90)
 		(descr "Resistor SMD 1206 (3216 Metric), square (rectangular) end terminal, IPC-7351 nominal with elongated pad for handsoldering. (Body size source: IPC-SM-782 page 72, https://www.pcb-3d.com/wordpress/wp-content/uploads/ipc-sm-782a_amendment_1_and_2.pdf), generated with kicad-footprint-generator")
 		(tags "resistor handsolder")
@@
 		(tags "connector JST XH vertical")
 		(property "Reference" "J7"
-			(at 1.25 3.55 180)
+			(at -3.8 2.275 180)
 			(layer "B.SilkS")
 			(effects
@@
 		(layer "Edge.Cuts")
 	)
+	(gr_text "UART"
+		(at 181.9 89.6 0)
+		(layer "F.SilkS" knockout)
+		(effects
+			(font
+				(size 0.75 0.75)
+				(thickness 0.15)
+				(bold yes)
+			)
+		)
+	)
 	(gr_text "Z"
-		(at 169 74.015 0)
+		(at 169 71.699999 0)
 		(layer "F.SilkS" knockout)
 		(effects
@@
 		)
 	)
-	(gr_text "Y"
+	(gr_text "B2-B1-A2-A1\nYEL-ORG-BLU-RED"
 		(at 150 74.015001 0)
 		(layer "F.SilkS" knockout)
@@
 		)
 	)
-	(gr_text "X"
+	(gr_text "B2-B1-A2-A1\nYEL-ORG-BLU-RED"
 		(at 131 74.015001 0)
 		(layer "F.SilkS" knockout)
@@
 		)
 	)
+	(gr_text "Y"
+		(at 150 71.7 0)
+		(layer "F.SilkS" knockout)
+		(effects
+			(font
+				(size 0.75 0.75)
+				(thickness 0.15)
+				(bold yes)
+			)
+			(justify bottom)
+		)
+	)
+	(gr_text "X"
+		(at 131 71.7 0)
+		(layer "F.SilkS" knockout)
+		(effects
+			(font
+				(size 0.75 0.75)
+				(thickness 0.15)
+				(bold yes)
+			)
+			(justify bottom)
+		)
+	)
+	(gr_text "B2-B1-A2-A1\nYEL-ORG-BLU-RED"
+		(at 169 74.015 0)
+		(layer "F.SilkS" knockout)
+		(effects
+			(font
+				(size 0.75 0.75)
+				(thickness 0.15)
+				(bold yes)
+			)
+			(justify bottom)
+		)
+	)
 	(gr_text "EXTERNAL\nPOWER"
 		(at 118.4 86.3 0)
@@
 		)
 	)
-	(gr_text "VPDS-R1"
+	(gr_text "GND"
+		(at 158.7 87.7 0)
+		(layer "F.SilkS" knockout)
+		(effects
+			(font
+				(size 0.75 0.75)
+				(thickness 0.15)
+				(bold yes)
+			)
+		)
+	)
+	(gr_text "VPDS-R2"
 		(at 178.267993 126.019816 0)
 		(layer "F.SilkS" knockout)
@@
 		)
 	)
+	(gr_text "+EXTERNAL"
+		(at 141.2 87.7 0)
+		(layer "F.SilkS" knockout)
+		(effects
+			(font
+				(size 0.75 0.75)
+				(thickness 0.15)
+				(bold yes)
+			)
+		)
+	)
+	(gr_text "+"
+		(at 145.9 127.5 0)
+		(layer "B.SilkS" knockout)
+		(effects
+			(font
+				(size 0.75 0.75)
+				(thickness 0.15)
+				(bold yes)
+			)
+			(justify mirror)
+		)
+	)
+	(gr_text "-"
+		(at 137.6 127.5 0)
+		(layer "B.SilkS" knockout)
+		(effects
+			(font
+				(size 0.75 0.75)
+				(thickness 0.15)
+				(bold yes)
+			)
+			(justify mirror)
+		)
+	)
+	(gr_text "+"
+		(at 128.9 127.5 0)
+		(layer "B.SilkS" knockout)
+		(effects
+			(font
+				(size 0.75 0.75)
+				(thickness 0.15)
+				(bold yes)
+			)
+			(justify mirror)
+		)
+	)
 	(gr_text "BATTERY-C"
 		(at 133.100001 123.5 0)
@@
 		)
 	)
+	(gr_text "+11V"
+		(at 132 130.7 0)
+		(layer "B.SilkS" knockout)
+		(effects
+			(font
+				(size 0.75 0.75)
+				(thickness 0.15)
+				(bold yes)
+			)
+			(justify mirror)
+		)
+	)
 	(gr_text "BATTERY-B"
 		(at 150.100001 123.4 0)
@@
 		)
 	)
+	(gr_text "-"
+		(at 171.6 127.5 0)
+		(layer "B.SilkS" knockout)
+		(effects
+			(font
+				(size 0.75 0.75)
+				(thickness 0.15)
+				(bold yes)
+			)
+			(justify mirror)
+		)
+	)
+	(gr_text "-"
+		(at 154.6 127.5 0)
+		(layer "B.SilkS" knockout)
+		(effects
+			(font
+				(size 0.75 0.75)
+				(thickness 0.15)
+				(bold yes)
+			)
+			(justify mirror)
+		)
+	)
 	(gr_text "BATTERY\nAS\nEXTERNAL"
 		(at 162.5 69.8 0)
@@
 		)
 	)
+	(gr_text "GND"
+		(at 168.5 130.7 0)
+		(layer "B.SilkS" knockout)
+		(effects
+			(font
+				(size 0.75 0.75)
+				(thickness 0.15)
+				(bold yes)
+			)
+			(justify mirror)
+		)
+	)
 	(gr_text "DISABLE\nBATTERY"
 		(at 150 70.7 0)
@@
 		)
 	)
+	(gr_text "WASTE PRODUCT\nOF\nPHUC DOAN"
+		(at 174.3 117.4 0)
+		(layer "B.SilkS" knockout)
+		(effects
+			(font
+				(size 1.5 1.5)
+				(thickness 0.375)
+				(bold yes)
+			)
+			(justify mirror)
+		)
+	)
 	(gr_text "DISABLE\nMOTORS"
 		(at 137.5 70.7 0)
@@
 		)
 	)
+	(gr_text "+"
+		(at 162.9 127.5 0)
+		(layer "B.SilkS" knockout)
+		(effects
+			(font
+				(size 0.75 0.75)
+				(thickness 0.15)
+				(bold yes)
+			)
+			(justify mirror)
+		)
+	)
 	(segment
 		(start 144.8 130.525)
@@
 	)
 	(segment
-		(start 127.6 132.2)
+		(start 127.3 132.2)
 		(end 147.1 132.2)
 		(width 0.2)
@@
 	)
 	(segment
-		(start 147.1 132.2)
-		(end 147.55 131.75)
+		(start 147.55 131.75)
+		(end 147.55 130.525)
 		(width 0.2)
 		(layer "F.Cu")
@@
 	)
 	(segment
-		(start 147.55 131.75)
-		(end 147.55 130.525)
+		(start 147.1 132.2)
+		(end 147.55 131.75)
 		(width 0.2)
 		(layer "F.Cu")
@@
 	)
 	(via
-		(at 127.6 132.2)
+		(at 127.3 132.2)
 		(size 0.6)
 		(drill 0.3)
@@
 	)
 	(segment
-		(start 127.6 132.2)
-		(end 127.6 127.4)
+		(start 127.3 132.2)
+		(end 127.3 127.4)
 		(width 0.2)
 		(layer "B.Cu")
@@
 	)
 	(segment
-		(start 126.3 123.1)
-		(end 127.5 124.3)
-		(width 0.2)
-		(layer "F.Cu")
-		(net 24)
-	)
-	(segment
 		(start 154.749999 67.5)
 		(end 154.8 67.449999)
@@
 	)
 	(segment
-		(start 127.5 124.3)
-		(end 132.3 124.3)
+		(start 126.1 123.1)
+		(end 117.3 123.1)
 		(width 0.2)
 		(layer "F.Cu")
@@
 	)
 	(segment
-		(start 154.8 67.449999)
-		(end 154.8 66.2)
+		(start 127.3 124.3)
+		(end 126.1 123.1)
 		(width 0.2)
 		(layer "F.Cu")
@@
 	)
 	(segment
-		(start 117.3 123.1)
-		(end 126.3 123.1)
+		(start 154.8 67.449999)
+		(end 154.8 66.2)
 		(width 0.2)
 		(layer "F.Cu")
@@
 		(net 24)
 	)
+	(segment
+		(start 127.3 124.3)
+		(end 132.3 124.3)
+		(width 0.2)
+		(layer "F.Cu")
+		(net 24)
+	)
 	(via
 		(at 117.3 123.1)
@@
 	)
 	(via
-		(at 127.5 124.3)
+		(at 127.3 124.3)
 		(size 0.6)
 		(drill 0.3)
