File: pcb/DebugBoard.kicad_sch (KiCad schematic)
At the start: 4 parts

Commit message: Basic expected components for `DebugBoard` PCB.
Parts:
- added BZ1: AST1109MLTRQ, Buzzer_Beeper:Buzzer_Mallory_AST1109MLTRQ, symbol Device:Buzzer
- added C1: 10u, Capacitor_SMD:C_1206_3216Metric_Pad1.33x1.80mm_HandSolder, symbol Device:C_Small
- added C2, C3, C5: 1u, Capacitor_SMD:C_1206_3216Metric_Pad1.33x1.80mm_HandSolder, symbol Device:C_Small
- added C4, C6: 100n, Capacitor_SMD:C_1206_3216Metric_Pad1.33x1.80mm_HandSolder, symbol Device:C_Small
- added C7: 10n, Capacitor_SMD:C_1206_3216Metric_Pad1.33x1.80mm_HandSolder, symbol Device:C_Small
- added D1, D2, D3, D4: 150141M173100, LED_SMD:LED_RGB_Wuerth-PLCC4_3.2x2.8mm_150141M173100, symbol Device:LED_ABRG
- added D5, D6, D8: GREEN, LED_SMD:LED_1206_3216Metric_Pad1.42x1.75mm_HandSolder, symbol Device:LED
- added D7: RED, LED_SMD:LED_1206_3216Metric_Pad1.42x1.75mm_HandSolder, symbol Device:LED
- added J1: Debug, pcb:Molex_PicoBlade_53047-1010_1x10_P1.25mm_Vertical, symbol Connector_Generic:Conn_01x10
- added J2: USB_C_Receptacle, pcb:USB_C_Receptacle_Amphenol_12401548E4-2A, symbol Connector:USB_C_Receptacle
- added J3: Conn_01x04, pcb:SSD1306_Module_Connector, symbol Connector_Generic:Conn_01x04
- added J4: B8B-XH-A, Connector_JST:JST_XH_B8B-XH-A_1x08_P2.50mm_Vertical, symbol Connector_Generic:Conn_01x08
- added J5: 0472192001, pcb:microSD_HC_Molex_47219-2001, symbol Connector:Micro_SD_Card
- added JP1: SolderJumper_2_Open, Jumper:SolderJumper-2_P1.3mm_Open_RoundedPad1.0x1.5mm, symbol Jumper:SolderJumper_2_Open
- added JP2: Jumper_3_Bridged12, Connector_PinHeader_2.54mm:PinHeader_1x03_P2.54mm_Vertical, symbol Jumper:Jumper_3_Bridged12
- added Q1: S8050, Package_TO_SOT_SMD:SOT-23_Handsoldering, symbol Transistor_BJT:S8050
- added R1: 5k1, Resistor_SMD:R_1206_3216Metric_Pad1.30x1.75mm_HandSolder, symbol Device:R
- added R10, R11, R12, R13, R14, R9: R_Small, Resistor_SMD:R_1206_3216Metric_Pad1.30x1.75mm_HandSolder, symbol Device:R_Small
- added R2, R4: 4K, Resistor_SMD:R_1206_3216Metric_Pad1.30x1.75mm_HandSolder, symbol Device:R
- added R3: 10K, Resistor_SMD:R_1206_3216Metric_Pad1.30x1.75mm_HandSolder, symbol Device:R
- added R5, R6: 2K, Resistor_SMD:R_1206_3216Metric_Pad1.30x1.75mm_HandSolder, symbol Device:R
- added R7: 50k, Resistor_SMD:R_1206_3216Metric_Pad1.30x1.75mm_HandSolder, symbol Device:R
- added R8: 10k, Resistor_SMD:R_1206_3216Metric_Pad1.30x1.75mm_HandSolder, symbol Device:R
- added SW1, SW2, SW3, SW4: B3U-1000P, Button_Switch_SMD:SW_SPST_B3U-1000P, symbol Switch:SW_Push
- added U1: STM32H533VET6, Package_QFP:LQFP-100_14x14mm_P0.5mm, symbol MCU_ST_STM32H5:STM32H533VETx
- added U2: MCP2221A-I/ST, Package_SO:TSSOP-14_4.4x5mm_P0.65mm, symbol Interface_USB:MCP2221AxST
- added U3: AP2112K-3.3, Package_TO_SOT_SMD:SOT-23-5, symbol Regulator_Linear:AP2112K-3.3
Connections:
- new net: D5.2 (A), R2.2
- new net: C1.1, C2.1, J2.A4 (VBUS), J2.A9 (VBUS), J2.B4 (VBUS), J2.B9 (VBUS), JP1.1 (A), R2.1, U3.1 (VIN)
- new net: J5.1 (DAT2), R9.2
- new net: J5.5 (CLK), R10.2
- new net: J5.2 (DAT3/CD), R11.2
- new net: D6.2 (A), R4.2
- new net: J5.7 (DAT0), R12.2
- new net: U1.10 (VSS), U1.27 (VSS), U1.49 (VSS), U1.74 (VSS), U1.99 (VSS)
- new net: D8.2 (A), R6.1
- new net: J5.3 (CMD), R13.2
- new net: D7.1 (K), U2.2 (GP0)
- new net: D7.2 (A), R5.2
- new net: J2.A5 (CC1), R1.2
- new net: J2.A6 (D+), J2.B6 (D+), U2.12 (D-)
- new net: J2.A7 (D-), J2.B7 (D-), U2.13 (D+)
- new net: JP2.1 (A), R8.1
- new net: JP2.3 (B), R7.1
- new net: J5.8 (DAT1), R14.2
- new net: D8.1 (K), U2.3 (GP1)
- new net: JP1.2 (B), U3.3 (EN)
- new net: Q1.2 (B), R7.2, R8.2
- new net: BZ1.2 (-), Q1.3 (C)
- new net +3.3V: BZ1.1 (+), C3.1, C4.1, C5.1, C6.1, C7.1, J1.1 (Pin_1), J3.2 (Pin_2), J4.1 (Pin_1), J5.4 (VDD), R3.1, R4.1, R5.1, R6.2, U2.1 (VDD), U2.11 (VUSB), U3.5 (VOUT)
- new net GND: C1.2, C2.2, C3.2, C4.2, C5.2, C6.2, C7.2, D5.1 (K), D6.1 (K), J1.10 (Pin_10), J1.5 (Pin_5), J1.6 (Pin_6), J2.A1 (GND), J2.A12 (GND), J2.B1 (GND), J2.B12 (GND), J2.S1 (SHIELD), J3.1 (Pin_1), J4.8 (Pin_8), J5.6 (VSS), J5.9 (SHIELD), Q1.1 (E), R1.1, U2.14 (VSS), U3.2 (GND)
- new net RESET: J1.2 (Pin_2)
- new net buzzer: JP2.2 (C)
- new net clock: R10.1
- new net cmd: R13.1
- new net data_0: R12.1
- new net data_1: R14.1
- new net data_2: R9.1
- new net data_3: R11.1
- new net debug_i2c_clock: J4.3 (Pin_3)
- new net debug_i2c_data: J4.2 (Pin_2)
- new net display_i2c_clock: J3.3 (Pin_3)
- new net display_i2c_data: J3.4 (Pin_4)
- new net serial_reset: R3.2, U2.4 (~{RST})
- new net serial_rx: U2.6 (UTx)
- new net serial_tx: U2.5 (URx)
- new net stlink_rx: J1.4 (Pin_4)
- new net stlink_tx: J1.3 (Pin_3)
- new net swclk: J1.7 (Pin_7)
- new net swdio: J1.8 (Pin_8)
- new net swo: J1.9 (Pin_9)
- no-connect marks 0 -> 15
Other:
- note added: "@/url:`community.st.com/t5/stm32-mcus-embedded-software/how-to-connect-the-cc-pin-when-make-usb-type-c-compatible-to/td-p/303605`."
- note added: "By factory default, GP0 signals URx activity, GP1 signals UTx activity, and they're both active-low. @/pg 3/tbl l-1/`MCP2221A`. @/pg 7/sec 1.4.2/`MCP2221A`."
- note added: "Convert the noisy 5V USB power to a (hopefully) clean 3.3V digital supply. The usage of AP2112 is taken from Adafruit's MCP2221A breakout board. @/pg 2/`AP2112`."
- note added: "Debug Buzzer (V6 : SMD Footprint)."
- note added: "Debug Connector (V2 : Removed To-Do)."
- note added: "Reference usage: @/url:`github.com/adafruit/Adafruit-MCP2221-PCB`."
- note added: "USB-UART Bridge (V8 : Enable with solder-bridge)."
- note added: "VDD and VUSB will be tied together. @/pg 18/fig 1-5/`MCP2221A`."
- note added: "serial_tx is where the MCU transmit the data and serial_rx is where the UART-bridge transmits the data that came from the PC."
- note added: "uSD Connector (V6 : Hierarchical labels)."
- moved on the sheet: H1, H2, H3, H4

Commit message: Worked out uSD connector and debug LEDs details for `DebugBoard`.
Parts:
- removed C5: 1u, Capacitor_SMD:C_1206_3216Metric_Pad1.33x1.80mm_HandSolder, symbol Device:C_Small
- removed C6: 100n, Capacitor_SMD:C_1206_3216Metric_Pad1.33x1.80mm_HandSolder, symbol Device:C_Small
- removed C7: 10n, Capacitor_SMD:C_1206_3216Metric_Pad1.33x1.80mm_HandSolder, symbol Device:C_Small
- removed D1, D2, D3, D4: 150141M173100, LED_SMD:LED_RGB_Wuerth-PLCC4_3.2x2.8mm_150141M173100, symbol Device:LED_ABRG
- removed J5: 0472192001, pcb:microSD_HC_Molex_47219-2001, symbol Connector:Micro_SD_Card
- removed R10, R11, R12, R13, R14, R9: R_Small, Resistor_SMD:R_1206_3216Metric_Pad1.30x1.75mm_HandSolder, symbol Device:R_Small
- added C10, C11, C12, C13, C14, C9: 100n, Capacitor_SMD:C_1206_3216Metric_Pad1.33x1.80mm_HandSolder, symbol Device:C_Small
- added C15, C16: 2u2, Capacitor_SMD:C_1206_3216Metric_Pad1.33x1.80mm_HandSolder, symbol Device:C_Small
- added C8: 4u7, Capacitor_SMD:C_1206_3216Metric_Pad1.33x1.80mm_HandSolder, symbol Device:C_Small
- added R15: 47k, Resistor_SMD:R_1206_3216Metric_Pad1.30x1.75mm_HandSolder, symbol Device:R
- added SW5: B3U-1000P, Button_Switch_SMD:SW_SPST_B3U-1000P, symbol Switch:SW_Push
Connections:
- net +3.3V: now also U1.100 (VDD), U1.11 (VDD), U1.21 (VREF+), U1.22 (VDDA), U1.28 (VDD), U1.50 (VDD), U1.6 (VBAT), U1.73 (VDDUSB), U1.75 (VDD), C10.1, C11.1, C12.1, C13.1, C14.1, C8.1, C9.1, SW5.1
- net GND: now also U1.10 (VSS), U1.19 (VSSA), U1.20 (VREF-), U1.27 (VSS), U1.49 (VSS), U1.74 (VSS), U1.99 (VSS), C10.2, C11.2, C12.2, C13.2, C14.2, C15.2, C16.2, C8.2, C9.2, R15.1
- net RESET: now also U1.14 (NRST)
- net buzzer: now also U1.30 (PA5)
- net serial_reset: now also U1.41 (PE10)
- net serial_rx: now also U1.58 (PD11)
- net serial_tx: now also U1.59 (PD12)
- net stlink_rx: now also U1.26 (PA3)
- net stlink_tx: now also U1.25 (PA2)
- net swclk: now also U1.76 (PA14(JTCK)
- net swdio: now also U1.72 (PA13(JTMS)
- net swo: now also U1.89 (PB3(JTDO)
- net vn100_sync_out: now reaches U1.12 (PH0)
- net led_channel_red: now reaches U1.15 (PC0)
- net led_channel_green: now reaches U1.16 (PC1)
- net openmv_spi_miso: now reaches U1.17 (PC2)
- net openmv_spi_mosi: now reaches U1.18 (PC3)
- net led_channel_blue: now reaches U1.23 (PA0)
- net motor_disable: now reaches U1.29 (PA4)
- net vn100_sync_in: now reaches U1.34 (PC5)
- net esp32_spi_miso: now reaches U1.35 (PB0)
- net esp32_spi_clock: now reaches U1.36 (PB1)
- net openmv_reset: now reaches U1.37 (PB2)
- net esp32_reset: now reaches U1.39 (PE8)
- net motor_step_z: now reaches U1.4 (PE5)
- net motor_step_x: now reaches U1.40 (PE9)
- net openmv_spi_clock: now reaches U1.47 (PB10)
- net VCAP: now reaches U1.48 (VCAP)
- net VCAP: now also U1.98 (VCAP), C15.1, C16.1
- net openmv_spi_nss: now reaches U1.51 (PB12)
- net motor_uart_tx: now reaches U1.53 (PB14)
- net motor_uart_rx: now reaches U1.54 (PB15)
- net vn100_uart_tx: now reaches U1.55 (PD8)
- net vn100_uart_rx: now reaches U1.56 (PD9)
- net lsm6dsv32x_interrupt_1: now reaches U1.60 (PD13)
- net lsm6dsv32x_interrupt_2: now reaches U1.61 (PD14)
- net lsm6dsv32x_chip_select: now reaches U1.62 (PD15)
- net motor_step_y: now reaches U1.63 (PC6)
- net sd_data_0: now reaches U1.65 (PC8)
- net sd_data_1: now reaches U1.66 (PC9)
- net motor_direction_y: now reaches U1.67 (PA8)
- net motor_direction_x: now reaches U1.68 (PA9)
- net motor_direction_z: now reaches U1.69 (PA10)
- net vn100_tare_restore: now reaches U1.7 (PC13)
- net sd_data_2: now reaches U1.78 (PC10)
- net sd_data_3: now reaches U1.79 (PC11)
- net sd_clock: now reaches U1.80 (PC12)
- net battery_allowed: now reaches U1.81 (PD0)
- net external_detected: now reaches U1.82 (PD1)
- net sd_cmd: now reaches U1.83 (PD2)
- net openmv_spi_ready: now reaches U1.86 (PD5)
- net vehicle_interface_i2c_clock: now reaches U1.87 (PD6)
- net vehicle_interface_i2c_data: now reaches U1.88 (PD7)
- net lis2mdl_chip_select: now reaches U1.9 (PC15)
- net lis2mdl_data_ready: now reaches U1.90 (PB4(NJTRST))
- net esp32_spi_mosi: now reaches U1.91 (PB5)
- net sensor_i2c_clock: now reaches U1.92 (PB6)
- net sensor_i2c_data: now reaches U1.93 (PB7)
- net BOOT0: now reaches U1.94 (BOOT0)
- net BOOT0: now also R15.2, SW5.2
- net esp32_spi_nss: now reaches U1.95 (PB8)
- net esp32_spi_ready: now reaches U1.97 (PE0)
- no-connect marks 15 -> 40
Other:
- added sheet RGB LED - A (DebugBoard_RGB_LED.kicad_sch)
- added sheet RGB LED - B (DebugBoard_RGB_LED.kicad_sch)
- added sheet RGB LED - C (DebugBoard_RGB_LED.kicad_sch)
- added sheet RGB LED - D (DebugBoard_RGB_LED.kicad_sch)
- added sheet uSD Connector (DebugBoard_uSD_Connector.kicad_sch)
- note added: ""If no external battery is used in the application, it is recommended to connect VBAT externally to VDD with a 100 nF external ceramic decoupling capacitor." @/pg 7/sec 2.1.4/`H533an`. "[VDDA] must be connected to VDD when these [analog] peripherals are not used." "[VDDUSB] must preferably be connected to VDD when the USB is not used." @/pg 3/sec 2.1/`H533an`."
- note added: ""If there are two VCAP pins (such as for the LQFP64 package), each pin must be connected to a 2.2uF (typical) capacitor (for a total approximately 4.4 uF)." @/pg 35/sec 8.2/`H533an`. @/pg 12/fig 6/`H533an`. @/pg 34/fig 14/`H533an`."
- note added: ""In addition, each power supply pair should be decoupled with filtering ceramic capacitors (100 nF) and one single ceramic capacitor (minimum 4.7 uF) connected in parallel." @/pg 31/sec 7.4/`H533an`."
- note added: "BOOT0 to GND has MCU boot from flash. @/pg 163/tbl 15/`H533rm`."
- note added: "STM32 MCU Support (V1 : Smaller BOOT0 setting)."
- note removed: "uSD Connector (V6 : Hierarchical labels)."
- moved on the sheet: BZ1, C1, C2, C3, C4, D5, D6, D7, D8, H1, H2, H3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
Changed lines of the file:
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@@
 	(generator "eeschema")
 	(generator_version "9.0")
-	(paper "A3")
+	(paper "A2")

Commit message: Added buttons and updated MCU pin-outs for `DebugBoard`.
Parts:
- removed J2: USB_C_Receptacle, pcb:USB_C_Receptacle_Amphenol_12401548E4-2A, symbol Connector:USB_C_Receptacle
- removed SW1, SW2, SW3, SW4: B3U-1000P, Button_Switch_SMD:SW_SPST_B3U-1000P, symbol Switch:SW_Push
- added J2: 12401598E4_2A, pcb:AMPHENOL_12401598E4_2A, symbol 12401598E4_2A:12401598E4_2A
- renumbered D5 to D2, D6 to D3, D7 to D4, D8 to D5
Connections:
- net esp32_reset is gone; now on net led_green_D: U1.39 (PE8)
- net esp32_spi_ready is gone; now on net led_red_B: U1.97 (PE0)
- net motor_direction_x is gone; now on net led_red_A: U1.68 (PA9)
- net motor_direction_z is gone; now on net led_green_A: U1.69 (PA10)
- net motor_step_x is gone; now on net led_blue_D: U1.40 (PE9)
- net motor_step_z is gone; now on net led_green_C: U1.4 (PE5)
- net sensor_i2c_clock is gone; now on net debug_i2c_clock: U1.92 (PB6)
- net sensor_i2c_data is gone; now on net debug_i2c_data: U1.93 (PB7)
- net vehicle_interface_i2c_clock is gone; now on net display_i2c_clock: U1.87 (PD6)
- net vehicle_interface_i2c_data is gone; now on net display_i2c_data: U1.88 (PD7)
- net +3.3V: now also J4.2 (Pin_2), J4.7 (Pin_7); no longer J4.1 (Pin_1)
- net GND: now also J4.1 (Pin_1), J2.A1 (GND), J2.A12 (GND__1), J2.B1 (GND__2), J2.B12 (GND__3), J2.SH1 (SHIELD), J2.SH2 (SHIELD__1), J2.SH3 (SHIELD__2), J2.SH4 (SHIELD__3)
- net debug_i2c_clock: now also J4.5 (Pin_5); no longer J4.3 (Pin_3)
- net debug_i2c_data: now also J4.4 (Pin_4); no longer J4.2 (Pin_2)
- net led_blue_A: now also U1.70 (PA11)
- net led_blue_B: now also U1.2 (PE3)
- net led_blue_C: now also U1.5 (PE6)
- net led_green_B: now also U1.1 (PE2)
- net led_red_C: now also U1.3 (PE4)
- net led_red_D: now also U1.38 (PE7)
- net at C1.1, C2.1, JP1.1 (A)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: now also J2.A4 (VBUS), J2.A9 (VBUS__1), J2.B4 (VBUS__2), J2.B9 (VBUS__3)
- net at R1.2: now also J2.A5 (CC1)
- net at U2.12 (D-): now also J2.A7 (DN1), J2.B7 (DN2)
- net at U2.13 (D+): now also J2.A6 (DP1), J2.B6 (DP2)
- net button_A: now reaches U1.42 (PE11)
- net button_B: now reaches U1.43 (PE12)
- net battery_allowed: no longer names the net of U1.81 (PD0)
- net esp32_spi_clock: no longer names the net of U1.36 (PB1)
- net esp32_spi_miso: no longer names the net of U1.35 (PB0)
- net esp32_spi_mosi: no longer names the net of U1.91 (PB5)
- net esp32_spi_nss: no longer names the net of U1.95 (PB8)
- net external_detected: no longer names the net of U1.82 (PD1)
- net led_channel_blue: no longer names the net of U1.23 (PA0)
- net led_channel_green: no longer names the net of U1.16 (PC1)
- net led_channel_red: no longer names the net of U1.15 (PC0)
- net lis2mdl_chip_select: no longer names the net of U1.9 (PC15)
- net lis2mdl_data_ready: no longer names the net of U1.90 (PB4(NJTRST))
- net lsm6dsv32x_chip_select: no longer names the net of U1.62 (PD15)
- net lsm6dsv32x_interrupt_1: no longer names the net of U1.60 (PD13)
- net lsm6dsv32x_interrupt_2: no longer names the net of U1.61 (PD14)
- net motor_direction_y: no longer names the net of U1.67 (PA8)
- net motor_disable: no longer names the net of U1.29 (PA4)
- net motor_step_y: no longer names the net of U1.63 (PC6)
- net motor_uart_rx: no longer names the net of U1.54 (PB15)
- net motor_uart_tx: no longer names the net of U1.53 (PB14)
- net openmv_reset: no longer names the net of U1.37 (PB2)
- net openmv_spi_clock: no longer names the net of U1.47 (PB10)
- net openmv_spi_miso: no longer names the net of U1.17 (PC2)
- net openmv_spi_mosi: no longer names the net of U1.18 (PC3)
- net openmv_spi_nss: no longer names the net of U1.51 (PB12)
- net openmv_spi_ready: no longer names the net of U1.86 (PD5)
- net vn100_sync_in: no longer names the net of U1.34 (PC5)
- net vn100_sync_out: no longer names the net of U1.12 (PH0)
- net vn100_tare_restore: no longer names the net of U1.7 (PC13)
- net vn100_uart_rx: no longer names the net of U1.56 (PD9)
- net vn100_uart_tx: no longer names the net of U1.55 (PD8)
- no-connect marks 40 -> 64
Other:
- added sheet Button - A (DebugBoard_Button.kicad_sch)
- added sheet Button - B (DebugBoard_Button.kicad_sch)
- note added: "USB-UART Bridge (V9 : Substituted receptacle)."
- note removed: "USB-UART Bridge (V8 : Enable with solder-bridge)."
- moved on the sheet: C1, C2, C3, C4, D2, D3, D4, D5, H1, H2, H3, H4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
