File: pcb/DebugBoard_RGB_LED.kicad_sch (KiCad schematic)
At the start: 4 parts

Commit message: Added buttons and updated MCU pin-outs for `DebugBoard`.
Changed lines of the file:
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@@
 	)
 	(hierarchical_label "blue_cathode"
-		(shape input)
+		(shape bidirectional)
 		(at 82.55 95.25 180)
 		(effects
@@
 	)
 	(hierarchical_label "red_cathode"
-		(shape input)
+		(shape bidirectional)
 		(at 82.55 77.47 180)
 		(effects
@@
 	)
 	(hierarchical_label "green_cathode"
-		(shape input)
+		(shape bidirectional)
 		(at 82.55 86.36 180)
 		(effects

Commit message: Made `DebugBoard` target and fixed some GPIO discrepancies.
Parts:
- renumbered R9 to R5, R10 to R6, R11 to R7
Changed lines of the file:
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@@
 		(dnp no)
 		(fields_autoplaced yes)
-		(property "Reference" "#PWR010"
+		(property "Reference" "#PWR030"
 			(at 102.87 63.5 0)
 			(effects
@@
 			(project "DebugBoard"
 				(path "/5ece3d0a-e9bb-4e6a-946b-805aaca75ace/40dfd0ae-dff4-4807-8e3f-21ef36050fce"
-					(reference "#PWR016")
-					(unit 1)
-				)
-				(path "/5ece3d0a-e9bb-4e6a-946b-805aaca75ace/cbacf443-23bd-449b-a54c-c7360b92e055"
-					(reference "#PWR011")
-					(unit 1)
-				)
-				(path "/5ece3d0a-e9bb-4e6a-946b-805aaca75ace/d153028f-6298-40d2-97f3-372782c46755"
-					(reference "#PWR015")
-					(unit 1)
-				)
-				(path "/5ece3d0a-e9bb-4e6a-946b-805aaca75ace/d47d76fd-7437-48e9-9697-c69b7824d8d5"
-					(reference "#PWR010")
+					(reference "#PWR033")
+					(unit 1)
+				)
+				(path "/5ece3d0a-e9bb-4e6a-946b-805aaca75ace/cbacf443-23bd-449b-a54c-c7360b92e055"
+					(reference "#PWR031")
+					(unit 1)
+				)
+				(path "/5ece3d0a-e9bb-4e6a-946b-805aaca75ace/d153028f-6298-40d2-97f3-372782c46755"
+					(reference "#PWR032")
+					(unit 1)
+				)
+				(path "/5ece3d0a-e9bb-4e6a-946b-805aaca75ace/d47d76fd-7437-48e9-9697-c69b7824d8d5"
+					(reference "#PWR030")
 					(unit 1)
 				)
@@
 		(dnp no)
 		(fields_autoplaced yes)
-		(property "Reference" "R9"
+		(property "Reference" "R5"
 			(at 95.25 72.3899 0)
 			(effects
@@
 			(project "DebugBoard"
 				(path "/5ece3d0a-e9bb-4e6a-946b-805aaca75ace/40dfd0ae-dff4-4807-8e3f-21ef36050fce"
-					(reference "R25")
-					(unit 1)
-				)
-				(path "/5ece3d0a-e9bb-4e6a-946b-805aaca75ace/cbacf443-23bd-449b-a54c-c7360b92e055"
-					(reference "R12")
-					(unit 1)
-				)
-				(path "/5ece3d0a-e9bb-4e6a-946b-805aaca75ace/d153028f-6298-40d2-97f3-372782c46755"
-					(reference "R22")
-					(unit 1)
-				)
-				(path "/5ece3d0a-e9bb-4e6a-946b-805aaca75ace/d47d76fd-7437-48e9-9697-c69b7824d8d5"
-					(reference "R9")
+					(reference "R14")
+					(unit 1)
+				)
+				(path "/5ece3d0a-e9bb-4e6a-946b-805aaca75ace/cbacf443-23bd-449b-a54c-c7360b92e055"
+					(reference "R8")
+					(unit 1)
+				)
+				(path "/5ece3d0a-e9bb-4e6a-946b-805aaca75ace/d153028f-6298-40d2-97f3-372782c46755"
+					(reference "R11")
+					(unit 1)
+				)
+				(path "/5ece3d0a-e9bb-4e6a-946b-805aaca75ace/d47d76fd-7437-48e9-9697-c69b7824d8d5"
+					(reference "R5")
 					(unit 1)
 				)
@@
 			(project "DebugBoard"
 				(path "/5ece3d0a-e9bb-4e6a-946b-805aaca75ace/40dfd0ae-dff4-4807-8e3f-21ef36050fce"
-					(reference "D11")
-					(unit 1)
-				)
-				(path "/5ece3d0a-e9bb-4e6a-946b-805aaca75ace/cbacf443-23bd-449b-a54c-c7360b92e055"
-					(reference "D9")
-					(unit 1)
-				)
-				(path "/5ece3d0a-e9bb-4e6a-946b-805aaca75ace/d153028f-6298-40d2-97f3-372782c46755"
-					(reference "D10")
+					(reference "D4")
+					(unit 1)
+				)
+				(path "/5ece3d0a-e9bb-4e6a-946b-805aaca75ace/cbacf443-23bd-449b-a54c-c7360b92e055"
+					(reference "D2")
+					(unit 1)
+				)
+				(path "/5ece3d0a-e9bb-4e6a-946b-805aaca75ace/d153028f-6298-40d2-97f3-372782c46755"
+					(reference "D3")
 					(unit 1)
 				)
@@
 		(dnp no)
 		(fields_autoplaced yes)
-		(property "Reference" "R10"
+		(property "Reference" "R6"
 			(at 100.33 81.2799 0)
 			(effects
@@
 			(project "DebugBoard"
 				(path "/5ece3d0a-e9bb-4e6a-946b-805aaca75ace/40dfd0ae-dff4-4807-8e3f-21ef36050fce"
-					(reference "R26")
-					(unit 1)
-				)
-				(path "/5ece3d0a-e9bb-4e6a-946b-805aaca75ace/cbacf443-23bd-449b-a54c-c7360b92e055"
-					(reference "R13")
-					(unit 1)
-				)
-				(path "/5ece3d0a-e9bb-4e6a-946b-805aaca75ace/d153028f-6298-40d2-97f3-372782c46755"
-					(reference "R23")
-					(unit 1)
-				)
-				(path "/5ece3d0a-e9bb-4e6a-946b-805aaca75ace/d47d76fd-7437-48e9-9697-c69b7824d8d5"
-					(reference "R10")
+					(reference "R15")
+					(unit 1)
+				)
+				(path "/5ece3d0a-e9bb-4e6a-946b-805aaca75ace/cbacf443-23bd-449b-a54c-c7360b92e055"
+					(reference "R9")
+					(unit 1)
+				)
+				(path "/5ece3d0a-e9bb-4e6a-946b-805aaca75ace/d153028f-6298-40d2-97f3-372782c46755"
+					(reference "R12")
+					(unit 1)
+				)
+				(path "/5ece3d0a-e9bb-4e6a-946b-805aaca75ace/d47d76fd-7437-48e9-9697-c69b7824d8d5"
+					(reference "R6")
 					(unit 1)
 				)
@@
 		(on_board yes)
 		(dnp no)
-		(property "Reference" "R11"
+		(property "Reference" "R7"
 			(at 105.41 90.1699 0)
 			(effects
@@
 			(project "DebugBoard"
 				(path "/5ece3d0a-e9bb-4e6a-946b-805aaca75ace/40dfd0ae-dff4-4807-8e3f-21ef36050fce"
-					(reference "R27")
-					(unit 1)
-				)
-				(path "/5ece3d0a-e9bb-4e6a-946b-805aaca75ace/cbacf443-23bd-449b-a54c-c7360b92e055"
-					(reference "R14")
-					(unit 1)
-				)
-				(path "/5ece3d0a-e9bb-4e6a-946b-805aaca75ace/d153028f-6298-40d2-97f3-372782c46755"
-					(reference "R24")
-					(unit 1)
-				)
-				(path "/5ece3d0a-e9bb-4e6a-946b-805aaca75ace/d47d76fd-7437-48e9-9697-c69b7824d8d5"
-					(reference "R11")
-					(unit 1)
-				)
+					(reference "R16")
+					(unit 1)
+				)
+				(path "/5ece3d0a-e9bb-4e6a-946b-805aaca75ace/cbacf443-23bd-449b-a54c-c7360b92e055"
+					(reference "R10")
+					(unit 1)
+				)
+				(path "/5ece3d0a-e9bb-4e6a-946b-805aaca75ace/d153028f-6298-40d2-97f3-372782c46755"
+					(reference "R13")
+					(unit 1)
+				)
+				(path "/5ece3d0a-e9bb-4e6a-946b-805aaca75ace/d47d76fd-7437-48e9-9697-c69b7824d8d5"
+					(reference "R7")
+					(unit 1)
+				)

Commit message: Placed silkscreen for `DebugBoard`.
Parts:
- renumbered D1 to D2, R5 to R1, R7 to R5
Changed lines of the file:
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@@
 		(dnp no)
 		(fields_autoplaced yes)
-		(property "Reference" "R5"
+		(property "Reference" "R1"
 			(at 95.25 72.3899 0)
 			(effects
@@
 			(project "DebugBoard"
 				(path "/5ece3d0a-e9bb-4e6a-946b-805aaca75ace/40dfd0ae-dff4-4807-8e3f-21ef36050fce"
-					(reference "R14")
+					(reference "R25")
 					(unit 1)
 				)
 				(path "/5ece3d0a-e9bb-4e6a-946b-805aaca75ace/cbacf443-23bd-449b-a54c-c7360b92e055"
-					(reference "R8")
+					(reference "R24")
 					(unit 1)
 				)
 				(path "/5ece3d0a-e9bb-4e6a-946b-805aaca75ace/d153028f-6298-40d2-97f3-372782c46755"
-					(reference "R11")
+					(reference "R4")
 					(unit 1)
 				)
 				(path "/5ece3d0a-e9bb-4e6a-946b-805aaca75ace/d47d76fd-7437-48e9-9697-c69b7824d8d5"
-					(reference "R5")
+					(reference "R1")
 					(unit 1)
 				)
@@
 		(dnp no)
 		(fields_autoplaced yes)
-		(property "Reference" "D1"
+		(property "Reference" "D2"
 			(at 111.76 63.4999 90)
 			(effects
@@
 			(project "DebugBoard"
 				(path "/5ece3d0a-e9bb-4e6a-946b-805aaca75ace/40dfd0ae-dff4-4807-8e3f-21ef36050fce"
-					(reference "D4")
+					(reference "D3")
 					(unit 1)
 				)
 				(path "/5ece3d0a-e9bb-4e6a-946b-805aaca75ace/cbacf443-23bd-449b-a54c-c7360b92e055"
+					(reference "D5")
+					(unit 1)
+				)
+				(path "/5ece3d0a-e9bb-4e6a-946b-805aaca75ace/d153028f-6298-40d2-97f3-372782c46755"
+					(reference "D1")
+					(unit 1)
+				)
+				(path "/5ece3d0a-e9bb-4e6a-946b-805aaca75ace/d47d76fd-7437-48e9-9697-c69b7824d8d5"
 					(reference "D2")
-					(unit 1)
-				)
-				(path "/5ece3d0a-e9bb-4e6a-946b-805aaca75ace/d153028f-6298-40d2-97f3-372782c46755"
-					(reference "D3")
-					(unit 1)
-				)
-				(path "/5ece3d0a-e9bb-4e6a-946b-805aaca75ace/d47d76fd-7437-48e9-9697-c69b7824d8d5"
-					(reference "D1")
 					(unit 1)
 				)
@@
 			(project "DebugBoard"
 				(path "/5ece3d0a-e9bb-4e6a-946b-805aaca75ace/40dfd0ae-dff4-4807-8e3f-21ef36050fce"
-					(reference "R15")
+					(reference "R23")
 					(unit 1)
 				)
 				(path "/5ece3d0a-e9bb-4e6a-946b-805aaca75ace/cbacf443-23bd-449b-a54c-c7360b92e055"
+					(reference "R17")
+					(unit 1)
+				)
+				(path "/5ece3d0a-e9bb-4e6a-946b-805aaca75ace/d153028f-6298-40d2-97f3-372782c46755"
 					(reference "R9")
-					(unit 1)
-				)
-				(path "/5ece3d0a-e9bb-4e6a-946b-805aaca75ace/d153028f-6298-40d2-97f3-372782c46755"
-					(reference "R12")
 					(unit 1)
 				)
@@
 		(on_board yes)
 		(dnp no)
-		(property "Reference" "R7"
+		(property "Reference" "R5"
 			(at 105.41 90.1699 0)
 			(effects
@@
 			(project "DebugBoard"
 				(path "/5ece3d0a-e9bb-4e6a-946b-805aaca75ace/40dfd0ae-dff4-4807-8e3f-21ef36050fce"
-					(reference "R16")
+					(reference "R22")
 					(unit 1)
 				)
 				(path "/5ece3d0a-e9bb-4e6a-946b-805aaca75ace/cbacf443-23bd-449b-a54c-c7360b92e055"
-					(reference "R10")
+					(reference "R18")
 					(unit 1)
 				)
 				(path "/5ece3d0a-e9bb-4e6a-946b-805aaca75ace/d153028f-6298-40d2-97f3-372782c46755"
-					(reference "R13")
+					(reference "R8")
 					(unit 1)
 				)
 				(path "/5ece3d0a-e9bb-4e6a-946b-805aaca75ace/d47d76fd-7437-48e9-9697-c69b7824d8d5"
-					(reference "R7")
-					(unit 1)
-				)
+					(reference "R5")
+					(unit 1)
+				)
