File: pcb/VehiclePowerDistributionSystem_Stepper_Motor_Driver_TMC2209.kicad_sch (KiCad schematic)
At the start: 16 parts, among them U4 TMC2209-LA-T

Commit message: Geographically reannotated `VehiclePowerDistributionSystem`.
Parts:
- renumbered C4 to C14, C2 to C17, C3 to C20, C5 to C21, C8 to C4, C7 to C5, C1 to C8, C6 to C9, D1 to D5, JP4 to JP5, JP3 to JP6, R4 to R11, R3 to R5, R5 to R8, TP2 to TP4, U4 to U3

Commit message: Deprecated `motor_uart_rx` for `VehicleFlightComputer` and `VehiclePowerDistributionSystem`.
Parts:
- renumbered C8 to C1, C17 to C2, C20 to C3, C14 to C4, C21 to C5, C9 to C6, C5 to C7, C4 to C8, D5 to D4, JP5 to JP7, R5 to R7, R11 to R8, R8 to R9, TP4 to TP3, U3 to U4

Commit message: Revised `VehiclePowerDistributionSystem`.
Parts:
- removed D4: YELLOW, LED_SMD:LED_1206_3216Metric_Pad1.42x1.75mm_HandSolder, symbol Device:LED
- removed JP6, JP7: SolderJumper_2_Open, Jumper:SolderJumper-2_P1.3mm_Open_RoundedPad1.0x1.5mm, symbol Jumper:SolderJumper_2_Open
- removed R7: 2k, Resistor_SMD:R_1206_3216Metric_Pad1.30x1.75mm_HandSolder, symbol Device:R
- removed TP3: TestPoint, TestPoint:TestPoint_Pad_1.0x1.0mm, symbol Connector:TestPoint
- renumbered C4 to C13, C2 to C16, C5 to C19, C3 to C20, C8 to C3, C7 to C4, C1 to C7, C6 to C8, R8 to R11, R9 to R8, U4 to U3
Connections:
- net DIR is gone; now on net GND: U3.19 (DIR)
- net STEP is gone; now on net GND: U3.16 (STEP)
- net VREF is gone; now on net +3.3V: U3.17 (VREF)
- net AD0: now reaches U3.9 (MS1/AD0)
- net AD1: now reaches U3.10 (MS2/AD1)
- net DISABLE renamed ENABLE
- net SPREAD: no longer names the net of U3.7 (SPREAD)
- no-connect marks 3 -> 5
Other:
- note removed: "TODO: Consult @/pg 17/sec 3.7/`TMC2209`."
- note removed: "TODO: Tests should be done on what happens if the stepper motors are turned."
