File: pcb/DebugBoard.kicad_pcb (KiCad board)
At the start: 4 copper layers, 50 x 50 mm, 72 parts, among them J1 Debug, J2 12401598E4_2A, J3 Conn_01x04, J4 B8B-XH-A, J5 0472192001, Q1 S8050, SW1 B3U-1000P, SW2 B3U-1000P, SW5 B3U-1000P, U1 STM32H533VET6, U2 MCP2221A-I/ST, U3 AP2112K-3.3

Commit message: Laid out and routed `DebugBoard`.
Parts:
- removed the C1 at (75.4, 67.5)
- removed the C2 at (75.4, 70.8)
- removed the C3 at (75.4, 74.2)
- removed the C4 at (75.4, 77.5)
- removed the D2 at (93.9, 87.6)
- removed the D3 at (93.9, 91.0)
- removed the D4 at (93.9, 94.4)
- removed the J2 at (150.0, 116.2)
- removed the JP1 at (92.6, 84.1)
- removed Q1: S8050, Package_TO_SOT_SMD:SOT-23_Handsoldering
- removed the R1 at (101.0, 112.0)
- removed the R16 at (105.6, 51.6)
- removed the R17 at (105.6, 54.9)
- removed the R18 at (105.6, 58.2)
- removed the R2 at (93.4, 70.7)
- removed the R5 at (93.4, 80.7)
- removed the R6 at (99.3, 67.4)
- removed the R8 at (99.3, 74.1)
- removed U2: MCP2221A-I/ST, Package_SO:TSSOP-14_4.4x5mm_P0.65mm
- removed U3: AP2112K-3.3, Package_TO_SOT_SMD:SOT-23-5
- added C13: 100n, Capacitor_SMD:C_1206_3216Metric_Pad1.33x1.80mm_HandSolder, B.Cu at (139.6, 77.5)
- added JP2: Jumper_2_Small_Bridged, TestPoint:TestPoint_2Pads_Pitch2.54mm_Drill0.8mm, F.Cu at (143.5, 83.1)
- added JP3: Jumper_2_Small_Bridged, TestPoint:TestPoint_2Pads_Pitch2.54mm_Drill0.8mm, F.Cu at (151.1, 83.1)
- added R22: 10k, Resistor_SMD:R_1206_3216Metric_Pad1.30x1.75mm_HandSolder, B.Cu at (131.6, 98.8)
- added R23: 10k, Resistor_SMD:R_1206_3216Metric_Pad1.30x1.75mm_HandSolder, B.Cu at (131.6, 101.3)
- added R24: 10k, Resistor_SMD:R_1206_3216Metric_Pad1.30x1.75mm_HandSolder, B.Cu at (131.6, 103.8)
- added R25: 10k, Resistor_SMD:R_1206_3216Metric_Pad1.30x1.75mm_HandSolder, B.Cu at (140.1, 122.0)
- added SW4: B3U-1000P, Button_Switch_SMD:SW_SPST_B3U-1000P, F.Cu at (140.7, 77.5)
- added TP1: TestPoint, TestPoint:TestPoint_Bridge_Pitch2.0mm_Drill0.7mm, F.Cu at (128.1, 114.9)
- added TP2: TestPoint, TestPoint:TestPoint_Bridge_Pitch2.0mm_Drill0.7mm, F.Cu at (128.1, 87.1)
- added TP3: TestPoint, TestPoint:TestPoint_Bridge_Pitch2.0mm_Drill0.7mm, F.Cu at (169.0, 114.5)
- added TP4: TestPoint, TestPoint:TestPoint_Bridge_Pitch2.0mm_Drill0.7mm, F.Cu at (167.5, 87.0)
- added TP5: TestPoint, TestPoint:TestPoint_Bridge_Pitch2.0mm_Drill0.7mm, F.Cu at (172.5, 87.0)
- added TP6: TestPoint, TestPoint:TestPoint_Bridge_Pitch2.0mm_Drill0.7mm, F.Cu at (170.0, 87.0)
- BZ1: moved to F.Cu
- C10: renamed from C17; moved to B.Cu
- C11: renamed from C18; moved to B.Cu
- C12: renamed from C19; moved to B.Cu
- R1: renamed from R15; moved to B.Cu
- R19: value R_Small -> 100; moved to B.Cu
- R2: renamed from R7; value 50k -> 10k; moved to B.Cu
- R20: value R_Small -> 1K; moved to B.Cu
- R21: value R_Small -> 10k; moved to B.Cu
- R3: value 10K -> 10k; moved to B.Cu
- R4: value 4K -> 10k; moved to B.Cu
- moved C10 79.5 mm to (147.6, 122.5), turned to -90 degrees
- moved C1 78.2 mm to (153.3, 101.5), turned to 135 degrees
- moved C2 78.0 mm to (155.0, 99.9), turned to 135 degrees
- moved C11 77.7 mm to (150.0, 122.5), turned to -90 degrees
- moved R4 76.2 mm to (154.7, 122.5), turned to 90 degrees
- moved C12 76.0 mm to (152.3, 122.5), turned to -90 degrees
- moved R2 74.0 mm to (170.0, 92.5), turned to 180 degrees
- moved C7 72.0 mm to (151.7, 103.2), turned to 135 degrees
- moved R3 71.0 mm to (145.3, 122.5), turned to 90 degrees
- moved C4 70.5 mm to (149.8, 98.0), turned to -45 degrees
- moved C8 69.8 mm to (150.1, 104.8), turned to 135 degrees
- moved C3 69.4 mm to (146.5, 101.2), turned to -45 degrees
- moved C5 68.5 mm to (148.2, 99.6), turned to -45 degrees
- moved JP1 68.3 mm to (167.5, 90.2), turned to 90 degrees
- moved C9 66.7 mm to (151.4, 96.3), turned to -45 degrees
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- renumbered C8 to C1, C9 to C2, C10 to C3, C11 to C4, C12 to C5, C13 to C6, C14 to C7, C15 to C8, C16 to C9, D9 to D2, D10 to D3, D11 to D4, J4 to J2, J5 to J4, JP2 to JP1, R14 to R10, R22 to R11, R23 to R12, R24 to R13, R25 to R14, R26 to R15, R27 to R16, R28 to R17, R29 to R18, R9 to R5, R10 to R6, R11 to R7, R12 to R8, R13 to R9, SW5 to SW1, SW1 to SW3
Connections:
- net debug_i2c_clock renamed communication_i2c_clock
- BZ1 pad 1: +3.3V -> Net-(BZ1-+)
- BZ1 pad 2: Net-(BZ1--) -> GND
- D5 pad 1: Net-(D5-K) -> GND
- J2 pad 3: unconnected-(J4-Pin_3-Pad3) -> communication_uart_rx_A
- J2 pad 4: debug_i2c_data -> communication_uart_rx_B
- J2 pad 6: unconnected-(J4-Pin_6-Pad6) -> communication_i2c_data
- J3 pad 1: GND -> Net-(J3-Pin_1)
- J3 pad 2: +3.3V -> Net-(J3-Pin_2)
- J4 pad 1: Net-(J5-DAT2) -> sd_data_2
- J4 pad 2: Net-(J5-DAT3/CD) -> sd_data_3
- J4 pad 3: Net-(J5-CMD) -> sd_cmd
- J4 pad 5: Net-(J5-CLK) -> sd_clock
- J4 pad 7: Net-(J5-DAT0) -> sd_data_0
- J4 pad 8: Net-(J5-DAT1) -> sd_data_1
- JP1 pad 1: Net-(JP2-A) -> Net-(BZ1-+)
- R10 pad 1: led_blue_C -> led_channel_blue_C
- R11 pad 1: led_red_B -> led_channel_red_B
- R12 pad 1: led_green_B -> led_channel_green_B
- R13 pad 1: led_blue_B -> led_channel_blue_B
- R14 pad 1: led_red_D -> led_channel_red_D
- R15 pad 1: led_green_D -> led_channel_green_D
- R16 pad 1: led_blue_D -> led_channel_blue_D
- R19 pad 1: sd_data_0 -> +3.3V
- R19 pad 2: Net-(J5-DAT0) -> RESET
- R2 pad 2: Net-(Q1-B) -> Net-(BZ1-+)
- R20 pad 1: sd_cmd -> Net-(R20-Pad1)
- R20 pad 2: Net-(J5-CMD) -> GND
- R21 pad 1: sd_data_1 -> communication_i2c_data
- R21 pad 2: Net-(J5-DAT1) -> +3.3V
- R3 pad 2: serial_reset -> sd_data_0
- R4 pad 2: Net-(D3-A) -> sd_cmd
- R5 pad 1: led_red_A -> led_channel_red_A
- R6 pad 1: led_green_A -> led_channel_green_A
- R7 pad 1: led_blue_A -> led_channel_blue_A
- R8 pad 1: led_red_C -> led_channel_red_C
- R9 pad 1: led_green_C -> led_channel_green_C
- U1 pad 1: led_green_B -> unconnected-(U1-PE2-Pad1)
- U1 pad 2: led_blue_B -> led_channel_red_A
- U1 pad 3: led_red_C -> led_channel_green_A
- U1 pad 32: unconnected-(U1-PA7-Pad32) -> led_channel_green_C
- U1 pad 33: unconnected-(U1-PC4-Pad33) -> led_channel_red_C
- U1 pad 34: unconnected-(U1-PC5-Pad34) -> led_channel_blue_C
- U1 pad 36: unconnected-(U1-PB1-Pad36) -> communication_uart_rx_B
- U1 pad 38: led_red_D -> unconnected-(U1-PE7-Pad38)
- U1 pad 39: led_green_D -> unconnected-(U1-PE8-Pad39)
- U1 pad 4: led_green_C -> led_channel_blue_A
- U1 pad 40: led_blue_D -> unconnected-(U1-PE9-Pad40)
- U1 pad 41: serial_reset -> /testpoint_A
- U1 pad 42: button_A -> unconnected-(U1-PE11-Pad42)
- U1 pad 45: unconnected-(U1-PE14-Pad45) -> button_A
- U1 pad 47: unconnected-(U1-PB10-Pad47) -> display_i2c_clock
- U1 pad 5: led_blue_C -> unconnected-(U1-PE6-Pad5)
- U1 pad 51: unconnected-(U1-PB12-Pad51) -> display_i2c_data
- U1 pad 54: unconnected-(U1-PB15-Pad54) -> communication_uart_rx_A
- U1 pad 58: serial_rx -> unconnected-(U1-PD11-Pad58)
- U1 pad 59: serial_tx -> unconnected-(U1-PD12-Pad59)
- U1 pad 68: led_red_A -> led_channel_red_D
- U1 pad 69: led_green_A -> led_channel_green_D
- U1 pad 70: led_blue_A -> led_channel_blue_D
- U1 pad 84: unconnected-(U1-PD3-Pad84) -> /testpoint_B
- U1 pad 85: unconnected-(U1-PD4-Pad85) -> led_channel_green_B
- U1 pad 86: unconnected-(U1-PD5-Pad86) -> led_channel_red_B
- U1 pad 87: display_i2c_clock -> led_channel_blue_B
- U1 pad 88: display_i2c_data -> unconnected-(U1-PD7-Pad88)
- U1 pad 93: debug_i2c_data -> communication_i2c_data
- U1 pad 97: led_red_B -> unconnected-(U1-PE0-Pad97)
Routing:
- net display_i2c_data: track 0.00 -> 49.7 mm, vias 0 -> 2
- net communication_uart_rx_B: track 0.00 -> 48.2 mm, vias 0 -> 4
- net swdio: track 0.00 -> 44.6 mm, vias 0 -> 3
- net display_i2c_clock: track 0.00 -> 42.9 mm, vias 0 -> 2
- net sd_cmd: track 0.00 -> 40.3 mm, vias 0 -> 2
- net /testpoint_A: track 0.00 -> 36.0 mm, vias 0 -> 2
- net RESET: track 0.00 -> 35.4 mm, vias 0 -> 2
- net sd_clock: track 0.00 -> 35.2 mm, vias 0 -> 1
- net stlink_rx: track 0.00 -> 34.8 mm, vias 0 -> 3
- net sd_data_3: track 0.00 -> 32.8 mm, vias 0 -> 1
- net swclk: track 0.00 -> 31.6 mm, vias 0 -> 3
- net sd_data_2: track 0.00 -> 30.9 mm, vias 0 -> 1
- net stlink_tx: track 0.00 -> 29.5 mm, vias 0 -> 3
- net led_channel_red_D: track 0.00 -> 28.3 mm, vias 0 -> 2
- net led_channel_red_C: track 0.00 -> 28.3 mm, vias 0 -> 2
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- added copper zone on B.Cu, net +3.3V
- added copper zone on F.Cu, net +3.3V
- added copper zone on In1.Cu, net GND
- added copper zone on In2.Cu, net GND
- removed copper zone on B.Cu, net (none)
- removed copper zone on F.Cu, net (none)
- removed copper zone on In1.Cu, net (none)
- removed copper zone on In2.Cu, net (none)

Commit message: Placed silkscreen for `DebugBoard`.
Parts:
- added G***: LOGO, LOGO, B.Cu at (142.8, 110.2)
- added G***: LOGO, LOGO, B.Cu at (150.7, 115.9)
- added G***: LOGO, LOGO, B.Cu at (168.2, 99.6)
- renumbered C6 to C1, C13 to C10, C12 to C11, C10 to C12, C11 to C13, C9 to C2, C2 to C6, C1 to C7, C7 to C9, D3 to D1, D1 to D2, D4 to D3, D5 to D4, D2 to D5, H3 to H1, H1 to H3, J3 to J2, J2 to J3, JP2 to JP1, JP3 to JP2, JP1 to JP3, R5 to R1, R2 to R10, R21 to R11, R22 to R12, R23 to R13, R24 to R14, R18 to R15, R17 to R16, R9 to R17, R10 to R18, R4 to R19, R1 to R2, R3 to R20, R25 to R21, R16 to R22, R15 to R23, R8 to R24, R14 to R25, R19 to R3, R11 to R4, R7 to R5, R20 to R7, R13 to R8, R12 to R9, SW4 to SW1, SW1 to SW2, SW2 to SW3, SW3 to SW4, TP2 to TP1, TP4 to TP2, TP6 to TP3, TP5 to TP4, TP1 to TP5, TP3 to TP6
Other:
- board text added: "+3.3V"
- board text added: "3.3V"
- board text added: "A"
- board text added: "B"
- board text added: "BOOT0"
- board text added: "BRAIN-WAVE RECORDING DEVICE"
- board text added: "C"
- board text added: "D"
- board text added: "DB-R1"
- board text added: "GND"
- board text added: "L"
- board text added: "Q"
- board text added: "RST"
- board text added: "RX_A"
- board text added: "RX_B"
- board text added: "SCL"
- board text added: "SDA"
- board text added: "SPACE-GRADE TRACKING PASSIVES"
- board text added: "WEAPON OF MASS SURVEILLANCE"

Commit message: Finalized `DB-R1`.
Changed lines of the file:
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@@
 		)
 	)
-	(gr_text "Q"
+	(gr_text "L"
 		(at 167.5 92.5 0)
 		(layer "F.SilkS" knockout)
@@
 		)
 	)
-	(gr_text "L"
+	(gr_text "Q"
 		(at 172.6 92.4 0)
 		(layer "F.SilkS" knockout)
