File: pcb/design.kicad_blocks/Timer_Event_Logic_Conversion.kicad_block/Timer_Event_Logic_Conversion.kicad_sch (KiCad schematic)
At the start: 4 parts

Commit message: Updated `Timer_Event_Logic_Conversion` design block.
Parts:
- removed C1: 1u, Capacitor_SMD:C_1206_3216Metric_Pad1.33x1.80mm_HandSolder, symbol Device:C
- added R17: 100k, Resistor_SMD:R_1206_3216Metric_Pad1.30x1.75mm_HandSolder, symbol Device:R
- D7: renamed from D4; value RED -> WHITE
- renumbered D5 to D8, R2 to R16
Connections:
- net GND: now also R17.2
- net INPUT: now also R17.1
Other:
- note added: "Acts as a drain for stray current."
- note added: "Timer Event Logic Conversion (V1 : Pull-down)."
- note removed: "Expected to draw 6.3mA - 9mA at 24V - 32V. Power disipated: 120mW - 241mW. Resistor that allows for the highest current to the zener without exceding its power rating. Note: Testing shows that zener can run at lower currents than specified on data sheet."
- note removed: "Timer Event Logic Conversion (V0)."
- moved on the sheet: D7, D8, R16
